File: kicad/kvm-atx.kicad_pcb (KiCad board)
At the start: 2 copper layers, 64.1 x 52.1 mm, 56 parts, among them J1 ATX, J2 I2C0, J3 UART0, K1 AQW210EHA, K2 AQW210EHA, SW1 RESET, SW2 POWER

Commit message: WIP assembly version
Parts:
- removed K1, K2: AQW210EHA, 000:SOP254P962X315-8N
- added U1: TLP172GM, 000:TLP172GM, F.Cu at (111.2, 46.2)
- added U2: TLP172GM, 000:TLP172GM, F.Cu at (111.4, 41.0)
- added U3: TLP172GM, 000:TLP172GM, F.Cu at (121.5, 69.0)
- added U4: TLP172GM, 000:TLP172GM, F.Cu at (121.5, 64.7)
- D3, D4: footprint LED_SMD:LED_1206_3216Metric_Pad1.42x1.75mm_HandSolder -> LED_SMD:LED_0603_1608Metric
- R1, R2, R3, R4, R5, R6: footprint Resistor_SMD:R_1206_3216Metric_Pad1.30x1.75mm_HandSolder -> Resistor_SMD:R_0603_1608Metric; moved to F.Cu
- R7, R8: footprint Resistor_SMD:R_1206_3216Metric_Pad1.30x1.75mm_HandSolder -> Resistor_SMD:R_0603_1608Metric
- moved R5 20.2 mm to (113.7, 66.4), turned to 90 degrees
- moved R6 10.6 mm to (107.0, 57.6), turned to 180 degrees
- moved R3 5.18 mm to (123.4, 61.1), turned to 0 degrees
- moved R4 0.43 mm to (123.3, 56.9), turned to 0 degrees
- turned R1 to 180 degrees
- turned R2 to 180 degrees
Routing:
- net Net-(U3-C): track 12.1 -> 1.87 mm, vias 1 -> 0
- net /GPIO14: track 30.9 -> 22.7 mm
- net /GPIO7: track 13.7 -> 6.88 mm
- net GND: track 8.43 -> 15.0 mm, vias 17 -> 19
- net /PWR_LED_P: track 3.31 -> 8.05 mm
- net Net-(U4-C): track 6.40 -> 1.84 mm, vias 1 -> 0
- net /GPIO15: track 25.8 -> 21.5 mm
- net Net-(U2-C): track 3.72 -> 0.00 mm, vias 1 -> 0
- net +3.3V: track 71.9 -> 73.9 mm
- net /PWR_LED_N: track 16.5 -> 14.9 mm
- net /HDD_LED_N: track 15.5 -> 14.2 mm, vias 0 -> 1
